File: Circuit/Main/FDC_Main.kicad_sch (KiCad schematic)
At the start: 37 parts, among them J3 I2C, J4 I2C, J5 Conn_01x07_Pin, J6 Fan, J7 100k, J8 Screw_Terminal_01x04, Q1 FDS6690A, Q2 T835-600B, U1 ATmega328-P, U2 MOC3043M, U3 SN74LVC2G06, Y1 16MHz

Commit message: Nested projects.
Other:
- note added: "Add snubber!"
Changed lines of the file:
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@@
+		)
+	)
+	(text "Add snubber!"
+		(exclude_from_sim no)
+		(at 281.178 131.572 0)
+		(effects
+			(font
+				(size 1.27 1.27)
+			)
 		)
 	)
