File: Circuit/Panel/FDC_Panel.kicad_sch (KiCad schematic)
At the start: 11 parts, among them J1 Interconnect, J2 Screen, SW1 Push

Commit message: Panel PCB almost done.
Changed lines of the file:
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@@
+	(wire
+		(pts
+			(xy 55.88 104.14) (xy 71.12 104.14)
+		)
+		(stroke
+			(width 0)
+			(type default)
+		)
+	)
 	(wire
 		(pts
@@
 	(wire
 		(pts
-			(xy 71.12 99.06) (xy 55.88 99.06)
-		)
-		(stroke
-			(width 0)
-			(type default)
-		)
-	)
-	(wire
-		(pts
 			(xy 110.49 80.01) (xy 110.49 74.93)
-		)
-		(stroke
-			(width 0)
-			(type default)
-		)
-	)
-	(wire
-		(pts
-			(xy 71.12 104.14) (xy 55.88 104.14)
 		)
 		(stroke
@@
 		)
 		(stroke
+			(width 0)
+			(type default)
+		)
+	)
+	(wire
+		(pts
+			(xy 55.88 99.06) (xy 71.12 99.06)
+		)
+		(stroke

Commit message: Nested projects.
Parts:
- renumbered H4 to H?, H1 to H?, H3 to H?, H2 to H?
Changed lines of the file:
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@@
 		(dnp no)
 		(fields_autoplaced yes)
-		(property "Reference" "#FLG01"
+		(property "Reference" "#FLG?"
 			(at 67.31 69.215 0)
 			(effects
@@
 		)
 		(instances
+			(project "FilamentDryerController"
+				(path "/aa35fc54-c042-44c0-931e-4bef950e8494/bb48b34f-e499-49be-8ddd-62ec4a8d0495"
+					(reference "#FLG?")
+					(unit 1)
+				)
+			)
 			(project "FDC_Panel"
 				(path "/ca11f4e8-dd1b-450f-82d2-0145ea9b47ab"
@@
 		(dnp no)
 		(fields_autoplaced yes)
-		(property "Reference" "H4"
+		(property "Reference" "H?"
 			(at 87.63 106.6799 0)
 			(effects
@@
 		)
 		(instances
+			(project "FilamentDryerController"
+				(path "/aa35fc54-c042-44c0-931e-4bef950e8494/bb48b34f-e499-49be-8ddd-62ec4a8d0495"
+					(reference "H?")
+					(unit 1)
+				)
+			)
 			(project "FDC_Panel"
 				(path "/ca11f4e8-dd1b-450f-82d2-0145ea9b47ab"
@@
 		(dnp no)
 		(fields_autoplaced yes)
-		(property "Reference" "#PWR04"
+		(property "Reference" "#PWR?"
 			(at 71.12 113.03 0)
 			(effects
@@
 		)
 		(instances
+			(project "FilamentDryerController"
+				(path "/aa35fc54-c042-44c0-931e-4bef950e8494/bb48b34f-e499-49be-8ddd-62ec4a8d0495"
+					(reference "#PWR?")
+					(unit 1)
+				)
+			)
 			(project "FDC_Panel"
 				(path "/ca11f4e8-dd1b-450f-82d2-0145ea9b47ab"
@@
 		(dnp no)
 		(fields_autoplaced yes)
-		(property "Reference" "H1"
+		(property "Reference" "H?"
 			(at 87.63 87.6299 0)
 			(effects
@@
 		)
 		(instances
+			(project "FilamentDryerController"
+				(path "/aa35fc54-c042-44c0-931e-4bef950e8494/bb48b34f-e499-49be-8ddd-62ec4a8d0495"
+					(reference "H?")
+					(unit 1)
+				)
+			)
 			(project ""
 				(path "/ca11f4e8-dd1b-450f-82d2-0145ea9b47ab"
@@
 		(dnp no)
 		(fields_autoplaced yes)
-		(property "Reference" "H3"
+		(property "Reference" "H?"
 			(at 87.63 100.3299 0)
 			(effects
@@
 		)
 		(instances
+			(project "FilamentDryerController"
+				(path "/aa35fc54-c042-44c0-931e-4bef950e8494/bb48b34f-e499-49be-8ddd-62ec4a8d0495"
+					(reference "H?")
+					(unit 1)
+				)
+			)
 			(project "FDC_Panel"
 				(path "/ca11f4e8-dd1b-450f-82d2-0145ea9b47ab"
@@
 		(dnp no)
 		(fields_autoplaced yes)
-		(property "Reference" "H2"
+		(property "Reference" "H?"
 			(at 87.63 93.9799 0)
 			(effects
@@
 		)
 		(instances
+			(project "FilamentDryerController"
+				(path "/aa35fc54-c042-44c0-931e-4bef950e8494/bb48b34f-e499-49be-8ddd-62ec4a8d0495"
+					(reference "H?")
+					(unit 1)
+				)
+			)
 			(project "FDC_Panel"
 				(path "/ca11f4e8-dd1b-450f-82d2-0145ea9b47ab"
@@
 		(dnp no)
 		(fields_autoplaced yes)
-		(property "Reference" "#PWR03"
+		(property "Reference" "#PWR?"
 			(at 71.12 100.33 0)
 			(effects
@@
 		)
 		(instances
+			(project "FilamentDryerController"
+				(path "/aa35fc54-c042-44c0-931e-4bef950e8494/bb48b34f-e499-49be-8ddd-62ec4a8d0495"
+					(reference "#PWR?")
+					(unit 1)
+				)
+			)
 			(project "FDC_Panel"
 				(path "/ca11f4e8-dd1b-450f-82d2-0145ea9b47ab"
@@
 		(dnp no)
 		(fields_autoplaced yes)
-		(property "Reference" "#FLG02"
+		(property "Reference" "#FLG?"
 			(at 73.025 73.66 0)
 			(effects
@@
 		)
 		(instances
-			(project "FDC_Panel"
-				(path "/ca11f4e8-dd1b-450f-82d2-0145ea9b47ab"
+			(project "FilamentDryerController"
+				(path "/aa35fc54-c042-44c0-931e-4bef950e8494/bb48b34f-e499-49be-8ddd-62ec4a8d0495"
+					(reference "#FLG?")
+					(unit 1)
+				)
+			)
+			(project "FDC_Panel"
+				(path "/ca11f4e8-dd1b-450f-82d2-0145ea9b47ab"
